File: PCB/EM7SEG_DRIVER_L9110S/EM7SEG_DRIVER.sch (KiCad schematic (older format))
At the start: 40 parts, among them J1 I2C_PWR_IN, J2 I2C_PWR_OUT, U1 EM7SEG, U2 MCP23017_SP, U3 L9110S, U4 L9110S, U5 L9110S, U6 L9110S, U7 L9110S, U8 L9110S, U9 L9110S

Commit message: use pull-downs instead of pull-ups for l9110 inputs
Parts:
- added J3: Pad_IO16, TestPoint:TestPoint_Pad_D1.0mm, symbol Connector:Conn_01x01_Male
Connections:
- net +5V: no longer R10.2, R11.2, R12.2, R13.2, R14.2, R15.2, R16.2, R17.2, R18.2, R19.2, R20.2, R21.2, R8.2, R9.2
- net GND: now also R10.2, R11.2, R12.2, R13.2, R14.2, R15.2, R16.2, R17.2, R18.2, R19.2, R20.2, R21.2, R8.2, R9.2
- net at U2.8 (GPB7): now also J3.1 (Pin_1)
- no-connect marks 3 -> 2
Other:
- note added: "Pulldowns for \nL9110S Inputs"
- note removed: "Pullups for \nL9110S Inputs"
- moved on the sheet: R10, R11, R12, R13, R14, R15, R16, R17, R18, R19, R20, R21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
